File: PowerLoad.kicad_sch (KiCad schematic)
At the start: 88 parts, among them IC1 L7812, J1 IN+, J2 IN-, J3 LOAD_IN+, J4 GND, J5 LOAD_IN+, U2 LM324, U3 LM324

Commit message: fixed super TO247-3
Parts:
- VD2, VD3, VD4, VD5: footprint Package_TO_SOT_THT:TO-247-3_Vertical -> SuperTO247-3:TO-247-3(powirtab)
Changed lines of the file:
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@@
 			)
 		)
-		(property "Footprint" "Package_TO_SOT_THT:TO-247-3_Vertical"
+		(property "Footprint" "SuperTO247-3:TO-247-3(powirtab)"
 			(at 39.37 148.59 90)
 			(effects
@@
 			)
 		)
-		(property "Footprint" "Package_TO_SOT_THT:TO-247-3_Vertical"
+		(property "Footprint" "SuperTO247-3:TO-247-3(powirtab)"
 			(at 39.37 137.16 90)
 			(effects
@@
 			)
 		)
-		(property "Footprint" "Package_TO_SOT_THT:TO-247-3_Vertical"
+		(property "Footprint" "SuperTO247-3:TO-247-3(powirtab)"
 			(at 39.37 170.18 90)
 			(effects
@@
 			)
 		)
-		(property "Footprint" "Package_TO_SOT_THT:TO-247-3_Vertical"
+		(property "Footprint" "SuperTO247-3:TO-247-3(powirtab)"
 			(at 39.37 158.75 90)
 			(effects
